Commit message: working on urdf

File: install/quadbot_nodes/share/quadbot_nodes/urdf/robot.urdf (robot description, URDF)
Before this commit: robot quadbot, 0 links, 0 joints
Links:
- added link base_link; collision box size=0.2 0.5 0.1; visual box size=0.2 0.5 0.1
- added link leg1_2joint; collision sphere radius=0.04; visual sphere radius=0.04
- added link leg1_2link; collision cylinder length=0.25 radius=0.03; visual cylinder length=0.25 radius=0.03
- added link leg1_3joint; collision sphere radius=0.04; visual sphere radius=0.04
- added link leg1_3link; collision cylinder length=0.02 radius=0.02; visual cylinder length=0.02 radius=0.02
- added link leg1_mainjoint; collision sphere radius=0.04; visual sphere radius=0.04
- added link leg1_mainlink; collision cylinder length=0.2 radius=0.03; visual cylinder length=0.25 radius=0.03
- added link leg1_wheel; collision cylinder length=0.035 radius=0.049; visual cylinder length=0.035 radius=0.049
Joints:
- added joint leg1_2Connection: type fixed, parent leg1_mainlink, child leg1_2joint, origin xyz=0 0 -0.5 rpy=0 0 0
- added joint leg1_2Rotation: type revolute, parent leg1_2joint, child leg1_2link, origin xyz=0 0 0 rpy=0 0 0, axis 0 0 1, limit lower=-1.57 upper=1.57 effort=10 velocity=1
- added joint leg1_3Connection: type fixed, parent leg1_2link, child leg1_3joint, origin xyz=0 0 -0.1 rpy=0 0 0
- added joint leg1_3Rotation: type revolute, parent leg1_3joint, child leg1_3link, origin xyz=0 0 0 rpy=0 0 0, axis 0 1 0, limit lower=-1.57 upper=1.57 effort=10 velocity=1
- added joint leg1_main: type fixed, parent base_link, child leg1_mainjoint, origin xyz=0.1 0.15 0.69 rpy=0 0 0
- added joint leg1_mainConnection: type revolute, parent leg1_mainjoint, child leg1_mainlink, origin xyz=0 0 0 rpy=0 0 0, axis 0 0 1, limit lower=-1.57 upper=1.57 effort=10 velocity=1
- added joint leg1_wheelConnection: type continuous, parent leg1_3link, child leg1_wheel, origin xyz=0 0 -0.02 rpy=-1.5707 0 -1.5707, axis 0 0 1

Commit message: first leg designed

File: install/quadbot_nodes/share/quadbot_nodes/urdf/robot.urdf (robot description, URDF)
Before this commit: robot quadbot, 8 links, 7 joints
Links:
- link leg1_3link: geometry collision cylinder length=0.07 radius=0.02; visual cylinder length=0.07 radius=0.02
Joints:
- joint leg1_2Connection: origin xyz=0 0 -0.5 rpy=0 0 0 -> xyz=0 0 -0.3 rpy=0 0 0
- joint leg1_2Rotation: axis 0 0 1 -> 1 0 0
- joint leg1_3Connection: origin xyz=0 0 -0.1 rpy=0 0 0 -> xyz=0 0 -0.28 rpy=0 0 0
- joint leg1_3Rotation: axis 0 1 0 -> 1 0 0
- joint leg1_mainConnection: axis 0 0 1 -> 1 0 0
- joint leg1_wheelConnection: origin xyz=0 0 -0.02 rpy=-1.5707 0 -1.5707 -> xyz=0 0 -0.13 rpy=-1.5707 0 -1.5707

Commit message: the 3 remaining arms were added + shoulders for the front arms

File: install/quadbot_nodes/share/quadbot_nodes/urdf/robot.urdf (robot description, URDF)
Before this commit: robot quadbot, 8 links, 7 joints
Links:
- added link leg1_shoulder; collision box size=0.08 0.08 0.08; visual box size=0.08 0.11 0.08
- added link leg2_2joint; collision sphere radius=0.04; visual sphere radius=0.04
- added link leg2_2link; collision cylinder length=0.25 radius=0.03; visual cylinder length=0.25 radius=0.03
- added link leg2_3joint; collision sphere radius=0.04; visual sphere radius=0.04
- added link leg2_3link; collision cylinder length=0.07 radius=0.02; visual cylinder length=0.07 radius=0.02
- added link leg2_mainjoint; collision sphere radius=0.04; visual sphere radius=0.04
- added link leg2_mainlink; collision cylinder length=0.2 radius=0.03; visual cylinder length=0.25 radius=0.03
- added link leg2_wheel; collision cylinder length=0.035 radius=0.049; visual cylinder length=0.035 radius=0.049
- added link leg3_2joint; collision sphere radius=0.04; visual sphere radius=0.04
- added link leg3_2link; collision cylinder length=0.25 radius=0.03; visual cylinder length=0.25 radius=0.03
- added link leg3_3joint; collision sphere radius=0.04; visual sphere radius=0.04
- added link leg3_3link; collision cylinder length=0.07 radius=0.02; visual cylinder length=0.07 radius=0.02
- added link leg3_mainjoint; collision sphere radius=0.04; visual sphere radius=0.04
- added link leg3_mainlink; collision cylinder length=0.2 radius=0.03; visual cylinder length=0.25 radius=0.03
- added link leg3_shoulder; collision box size=0.08 0.08 0.08; visual box size=0.08 0.11 0.08
- added link leg3_wheel; collision cylinder length=0.035 radius=0.049; visual cylinder length=0.035 radius=0.049
- added link leg4_2joint; collision sphere radius=0.04; visual sphere radius=0.04
- added link leg4_2link; collision cylinder length=0.25 radius=0.03; visual cylinder length=0.25 radius=0.03
- added link leg4_3joint; collision sphere radius=0.04; visual sphere radius=0.04
- added link leg4_3link; collision cylinder length=0.07 radius=0.02; visual cylinder length=0.07 radius=0.02
- added link leg4_mainjoint; collision sphere radius=0.04; visual sphere radius=0.04
- added link leg4_mainlink; collision cylinder length=0.2 radius=0.03; visual cylinder length=0.25 radius=0.03
- added link leg4_wheel; collision cylinder length=0.035 radius=0.049; visual cylinder length=0.035 radius=0.049
Joints:
- added joint leg1_shoulderConnection: type fixed, parent base_link, child leg1_shoulder, origin xyz=0.1 0.15 0.69 rpy=0 0 0
- added joint leg2_2Connection: type fixed, parent leg2_mainlink, child leg2_2joint, origin xyz=0 0 -0.3 rpy=0 0 0
- added joint leg2_2Rotation: type revolute, parent leg2_2joint, child leg2_2link, origin xyz=0 0 0 rpy=0 0 0, axis 1 0 0, limit lower=-1.57 upper=1.57 effort=10 velocity=1
- added joint leg2_3Connection: type fixed, parent leg2_2link, child leg2_3joint, origin xyz=0 0 -0.28 rpy=0 0 0
- added joint leg2_3Rotation: type revolute, parent leg2_3joint, child leg2_3link, origin xyz=0 0 0 rpy=0 0 0, axis 1 0 0, limit lower=-1.57 upper=1.57 effort=10 velocity=1
- added joint leg2_main: type fixed, parent base_link, child leg2_mainjoint, origin xyz=0.1 -0.15 0.69 rpy=0 0 0
- added joint leg2_mainConnection: type revolute, parent leg2_mainjoint, child leg2_mainlink, origin xyz=0 0 0 rpy=0 0 0, axis 1 0 0, limit lower=-1.57 upper=0.8 effort=10 velocity=1
- added joint leg2_wheelConnection: type continuous, parent leg2_3link, child leg2_wheel, origin xyz=0 0 -0.13 rpy=-1.5707 0 -1.5707, axis 0 0 1
- added joint leg3_2Connection: type fixed, parent leg3_mainlink, child leg3_2joint, origin xyz=0 0 -0.3 rpy=0 0 0
- added joint leg3_2Rotation: type revolute, parent leg3_2joint, child leg3_2link, origin xyz=0 0 0 rpy=0 0 0, axis 1 0 0, limit lower=-1.57 upper=1.57 effort=10 velocity=1
- added joint leg3_3Connection: type fixed, parent leg3_2link, child leg3_3joint, origin xyz=0 0 -0.28 rpy=0 0 0
- added joint leg3_3Rotation: type revolute, parent leg3_3joint, child leg3_3link, origin xyz=0 0 0 rpy=0 0 0, axis 1 0 0, limit lower=-1.57 upper=1.57 effort=10 velocity=1
- added joint leg3_main: type fixed, parent leg3_shoulder, child leg3_mainjoint, origin xyz=-0.06 0.04 0 rpy=0 0 0
- added joint leg3_mainConnection: type revolute, parent leg3_mainjoint, child leg3_mainlink, origin xyz=0 0 0 rpy=0 0 0, axis 1 0 0, limit lower=-1.57 upper=1.57 effort=10 velocity=1
- added joint leg3_shoulderConnection: type fixed, parent base_link, child leg3_shoulder, origin xyz=-0.1 0.15 0.69 rpy=0 0 0
- added joint leg3_wheelConnection: type continuous, parent leg3_3link, child leg3_wheel, origin xyz=0 0 -0.13 rpy=-1.5707 0 -1.5707, axis 0 0 1
- added joint leg4_2Connection: type fixed, parent leg4_mainlink, child leg4_2joint, origin xyz=0 0 -0.3 rpy=0 0 0
- added joint leg4_2Rotation: type revolute, parent leg4_2joint, child leg4_2link, origin xyz=0 0 0 rpy=0 0 0, axis 1 0 0, limit lower=-1.57 upper=1.57 effort=10 velocity=1
- added joint leg4_3Connection: type fixed, parent leg4_2link, child leg4_3joint, origin xyz=0 0 -0.28 rpy=0 0 0
- added joint leg4_3Rotation: type revolute, parent leg4_3joint, child leg4_3link, origin xyz=0 0 0 rpy=0 0 0, axis 1 0 0, limit lower=-1.57 upper=1.57 effort=10 velocity=1
- added joint leg4_main: type fixed, parent base_link, child leg4_mainjoint, origin xyz=-0.1 -0.15 0.69 rpy=0 0 0
- added joint leg4_mainConnection: type revolute, parent leg4_mainjoint, child leg4_mainlink, origin xyz=0 0 0 rpy=0 0 0, axis 1 0 0, limit lower=-1.57 upper=0.8 effort=10 velocity=1
- added joint leg4_wheelConnection: type continuous, parent leg4_3link, child leg4_wheel, origin xyz=0 0 -0.13 rpy=-1.5707 0 -1.5707, axis 0 0 1
- joint leg1_main: origin xyz=0.1 0.15 0.69 rpy=0 0 0 -> xyz=0.06 0.04 0 rpy=0 0 0; parent base_link -> leg1_shoulder

Commit message: added gazebo sim and ros2_controllers to controll joints

File: install/quadbot_nodes/share/quadbot_nodes/urdf/robot.urdf (robot description, URDF)
Before this commit: robot quadbot, 31 links, 30 joints
Links:
- link base_link: mass None -> 2.0
- link leg1_2joint: mass None -> 0.05
- link leg1_2link: mass None -> 0.3
- link leg1_3joint: mass None -> 0.05
- link leg1_3link: mass None -> 0.05
- link leg1_mainjoint: mass None -> 0.05
- link leg1_mainlink: mass None -> 0.3
- link leg1_shoulder: mass None -> 0.2
- link leg1_wheel: mass None -> 0.1
- link leg2_2joint: mass None -> 0.05
- link leg2_2link: mass None -> 0.3
- link leg2_3joint: mass None -> 0.05
- link leg2_3link: mass None -> 0.05
- link leg2_mainjoint: mass None -> 0.05
- link leg2_mainlink: mass None -> 0.3
- link leg2_wheel: mass None -> 0.1
- link leg3_2joint: mass None -> 0.05
- link leg3_2link: mass None -> 0.3
- link leg3_3joint: mass None -> 0.05
- link leg3_3link: mass None -> 0.05
- link leg3_mainjoint: mass None -> 0.05
- link leg3_mainlink: mass None -> 0.3
- link leg3_shoulder: mass None -> 0.2
- link leg3_wheel: mass None -> 0.1
- link leg4_2joint: mass None -> 0.05
- link leg4_2link: mass None -> 0.3
- link leg4_3joint: mass None -> 0.05
- link leg4_3link: mass None -> 0.05
- link leg4_mainjoint: mass None -> 0.05
- link leg4_mainlink: mass None -> 0.3
- link leg4_wheel: mass None -> 0.1
